Commit message: Added ROS Control/Hardware Interface/Joint Config

File: dtb_quadruped/dtb_quadruped_description/robots/dtb_quadruped.gazebo.xacro (robot description, xacro)
@@ -1,4 +1,24 @@
 <?xml version="1.0"?>
 <robot xmlns:xacro="http://ros.org/wiki/xacro" name="dtb_quadruped">
+	<!-- ROS Control Plugin -->
+	<gazebo>
+		<plugin name="gazebo_ros_control" filename="libgazebo_ros_control.so">
+		<robotNamespace>/dtb_quadruped</robotNamespace>
+		<robotSimType>gazebo_ros_control/DefaultRobotHWSim</robotSimType>
+		</plugin>
+	</gazebo>
+	<!-- Macro for Material properties -->
+	<xacro:macro name="material_prop_macro" params="link_name">
+		<gazebo reference="${link_name}">
+			<kp>1000.0</kp>
+			<kd>1000.0</kd>
+			<mu1>10.0</mu1>
+			<mu2>10.0</mu2>
+		</gazebo>
+	</xacro:macro>
+	<xacro:material_prop_macro link_name="calf_semicirc_1_1"/>
+	<xacro:material_prop_macro link_name="calf_semicirc_2_1"/>
+	<xacro:material_prop_macro link_name="calf_semicirc_2_1"/>
+	<xacro:material_prop_macro link_name="calf_semicirc_2_1"/>
 	<!-- Gazebo Colors -->
 	<xacro:macro name="white_color_macro" params="link_name">

File: dtb_quadruped/dtb_quadruped_description/robots/dtb_quadruped.urdf.xacro (robot description, xacro)
@@ -335,4 +335,29 @@
 	<xacro:calf_semicirc_macro calf_num="4" up_down="-1"/>
 	<xacro:calf_semicirc_macro calf_num="4" up_down="1"/>
+	<!-- Hardware Transmission -->
+	<xacro:macro name="transmission_macro" params="link_name">
+		<transmission name="${link_name}_transmission">
+			<type>transmission_interface/SimpleTransmission</type>
+			<joint name="${link_name}_joint">
+				<hardwareInterface>hardware_interface/EffortJointInterface</hardwareInterface>
+			</joint>
+			<actuator name="${link_name}_actuator">
+				<hardwareInterface>hardware_interface/EffortJointInterface</hardwareInterface>
+				<mechanicalReduction>1</mechanicalReduction>
+			</actuator>
+		</transmission>
+	</xacro:macro>
+	<xacro:transmission_macro link_name="t_motor_1"/>
+	<xacro:transmission_macro link_name="t_motor_2"/>
+	<xacro:transmission_macro link_name="t_motor_3"/>
+	<xacro:transmission_macro link_name="t_motor_4"/>
+	<xacro:transmission_macro link_name="l_motor_1"/>
+	<xacro:transmission_macro link_name="l_motor_2"/>
+	<xacro:transmission_macro link_name="l_motor_3"/>
+	<xacro:transmission_macro link_name="l_motor_4"/>
+	<xacro:transmission_macro link_name="h_motor_1"/>
+	<xacro:transmission_macro link_name="h_motor_2"/>
+	<xacro:transmission_macro link_name="h_motor_3"/>
+	<xacro:transmission_macro link_name="h_motor_4"/>
 	<!-- Rviz Colors -->
 	<material name = "body_color">

Commit message: Fixed friction and pid issues

File: dtb_quadruped/dtb_quadruped_description/robots/dtb_quadruped.gazebo.xacro (robot description, xacro)
@@ -9,16 +9,55 @@
 	</gazebo>
 	<!-- Macro for Material properties -->
-	<xacro:macro name="material_prop_macro" params="link_name">
+	<xacro:macro name="foot_material_prop_macro" params="link_name">
 		<gazebo reference="${link_name}">
-			<kp>1000.0</kp>
-			<kd>1000.0</kd>
+			<kp>100000.0</kp>
+			<kd>100000.0</kd>
 			<mu1>10.0</mu1>
 			<mu2>10.0</mu2>
+			<selfCollide>false</selfCollide>
 		</gazebo>
 	</xacro:macro>
-	<xacro:material_prop_macro link_name="calf_semicirc_1_1"/>
-	<xacro:material_prop_macro link_name="calf_semicirc_2_1"/>
-	<xacro:material_prop_macro link_name="calf_semicirc_2_1"/>
-	<xacro:material_prop_macro link_name="calf_semicirc_2_1"/>
+	<xacro:foot_material_prop_macro link_name="calf_semicirc_1_-1"/>
+	<xacro:foot_material_prop_macro link_name="calf_semicirc_2_-1"/>
+	<xacro:foot_material_prop_macro link_name="calf_semicirc_3_-1"/>
+	<xacro:foot_material_prop_macro link_name="calf_semicirc_4_-1"/>
+	<xacro:macro name="body_material_prop_macro" params="link_name">
+		<gazebo reference="${link_name}">
+			<kp>100000.0</kp>
+			<kd>100000.0</kd>
+			<mu1>0.5</mu1>
+			<mu2>0.5</mu2>
+			<selfCollide>false</selfCollide>
+		</gazebo>
+	</xacro:macro>
+	<xacro:body_material_prop_macro link_name="base_link"/>
+	<xacro:body_material_prop_macro link_name="t_motor_1"/>
+	<xacro:body_material_prop_macro link_name="t_motor_2"/>
+	<xacro:body_material_prop_macro link_name="t_motor_3"/>
+	<xacro:body_material_prop_macro link_name="t_motor_4"/>
+	<xacro:body_material_prop_macro link_name="l_motor_1"/>
+	<xacro:body_material_prop_macro link_name="l_motor_2"/>
+	<xacro:body_material_prop_macro link_name="l_motor_3"/>
+	<xacro:body_material_prop_macro link_name="l_motor_4"/>
+	<xacro:body_material_prop_macro link_name="h_motor_1"/>
+	<xacro:body_material_prop_macro link_name="h_motor_2"/>
+	<xacro:body_material_prop_macro link_name="h_motor_3"/>
+	<xacro:body_material_prop_macro link_name="h_motor_4"/>
+	<xacro:body_material_prop_macro link_name="t_l_link_1"/>
+	<xacro:body_material_prop_macro link_name="t_l_link_2"/>
+	<xacro:body_material_prop_macro link_name="t_l_link_3"/>
+	<xacro:body_material_prop_macro link_name="t_l_link_4"/>
+	<xacro:body_material_prop_macro link_name="thigh_link_1"/>
+	<xacro:body_material_prop_macro link_name="thigh_link_2"/>
+	<xacro:body_material_prop_macro link_name="thigh_link_3"/>
+	<xacro:body_material_prop_macro link_name="thigh_link_4"/>
+	<xacro:body_material_prop_macro link_name="calf_link_1"/>
+	<xacro:body_material_prop_macro link_name="calf_link_2"/>
+	<xacro:body_material_prop_macro link_name="calf_link_3"/>
+	<xacro:body_material_prop_macro link_name="calf_link_4"/>
+	<xacro:body_material_prop_macro link_name="calf_semicirc_1_1"/>
+	<xacro:body_material_prop_macro link_name="calf_semicirc_2_1"/>
+	<xacro:body_material_prop_macro link_name="calf_semicirc_3_1"/>
+	<xacro:body_material_prop_macro link_name="calf_semicirc_4_1"/>
 	<!-- Gazebo Colors -->
 	<xacro:macro name="white_color_macro" params="link_name">

File: dtb_quadruped/dtb_quadruped_description/robots/dtb_quadruped.urdf.xacro (robot description, xacro)
@@ -6,6 +6,7 @@
 	<xacro:property name="body_box_width" value="0.25"/>
 	<xacro:property name="body_box_height" value="0.1"/>
-	<xacro:property name="M_PI" value="3.1415926535897931"/>
-	<xacro:property name="motor_effort" value="30"/>
+	<xacro:property name="M_PI" value="3.1415926"/>
+	<xacro:property name="motor_effort" value="50"/>
+	<xacro:property name="motor_velocity" value="${M_PI/2}"/>
 	<!-- Base Description-->
 	<link name="base_footprint"/>
@@ -32,9 +33,9 @@
 		<inertial>
 			<origin xyz = "0 0 0" rpy = "0 0 0"/>
-			<mass value = "2.0"/>
+			<mass value = "4.0"/>
 			<inertia
-    	    	ixx="0.01201" ixy="0.0" ixz="0.0"
-    	    	iyy="0.06167" iyz="0.0"
-    	    	izz="0.07042"/>
+    	    	ixx="0.002201" ixy="0.0" ixz="0.0"
+    	    	iyy="0.008167" iyz="0.0"
+    	    	izz="0.009042"/>
 		</inertial>
 	</link>
@@ -69,5 +70,5 @@
 			<origin xyz="${x_pos} ${((body_box_width/2)-0.03)*y_pos} ${(-body_box_height/2)+0.04}" rpy="0 ${M_PI/2} 0"/>
 			<axis xyz="0 0 1"/>
-			<limit effort="${motor_effort}" lower="${(-M_PI/10)*y_pos}" upper="${(M_PI/10)*y_pos}" velocity="157"/>
+			<limit effort="${motor_effort}" lower="${-(M_PI/10)}" upper="${(M_PI/10)}" velocity="${motor_velocity}"/>
 		</joint>
 	</xacro:macro>
@@ -142,5 +143,5 @@
 			<origin xyz="0 ${(0.055)*pose} 0" rpy="${(-M_PI/2)*pose} 0 0"/>
 			<axis xyz="0 0 1"/>
-			<limit effort="${motor_effort}" lower="${(-M_PI/2)+((-M_PI/2)*pose)}" upper="${(M_PI/2)-((M_PI/2)*pose)}" velocity="157"/>
+			<limit effort="${motor_effort}" lower="${(-M_PI/2)+((-M_PI/2)*pose)}" upper="${(M_PI/2)-((M_PI/2)*pose)}" velocity="${motor_velocity}"/>
 		</joint>
 	</xacro:macro>
@@ -167,9 +168,9 @@
 			<inertial>
 				<origin xyz = "0 0 0" rpy = "0 0 0"/>
-				<mass value = "0.3"/>
-				<inertia
-    	    			ixx="0.0001825" ixy="0.0" ixz="0.0"
-    	    			iyy="0.001585" iyz="0.0"
-    	    			izz="0.001722"/>
+				<mass value = "0.5"/>
+				<inertia
+    	    			ixx="0.0002825" ixy="0.0" ixz="0.0"
+    	    			iyy="0.002585" iyz="0.0"
+    	    			izz="0.002722"/>
 			</inertial>
 		</link>
@@ -194,18 +195,4 @@
 				<material name = "thigh_color"/>
 			</visual>
-			<collision>
-				<origin xyz = "0 0 0" rpy = "0 0 0"/>
-				<geometry>
-					<cylinder length="0.03" radius="0.04"/>
-				</geometry>
-			</collision>
-			<inertial>
-				<origin xyz = "0 0 0" rpy = "0 0 0"/>
-				<mass value = "0.1"/>
-				<inertia
-    	    			ixx="0.0000475" ixy="0.0" ixz="0.0"
-    	    			iyy="0.0000475" iyz="0.0"
-    	    			izz="0.00008"/>
-			</inertial>
 		</link>
 		<joint name="thigh_semicirc_${thigh_num}_${up_down}_joint" type="fixed">
@@ -254,5 +241,5 @@
 			<origin xyz="0.125 0 0.015" rpy="0 0 0"/>
 			<axis xyz="0 0 1"/>
-			<limit effort="${motor_effort}" lower="${0 + (-M_PI*pose)}" upper="${M_PI-(pose*M_PI)}" velocity="157"/>
+			<limit effort="${motor_effort}" lower="${0 + (-M_PI*pose)}" upper="${M_PI-(pose*M_PI)}" velocity="${motor_velocity}"/>
 		</joint>
 	</xacro:macro>
@@ -279,9 +266,9 @@
 			<inertial>
 				<origin xyz = "0 0 0" rpy = "0 0 0"/>
-				<mass value = "0.3"/>
-				<inertia
-    	    			ixx="0.0001825" ixy="0.0" ixz="0.0"
-    	    			iyy="0.001585" iyz="0.0"
-    	    			izz="0.001722"/>
+				<mass value = "0.5"/>
+				<inertia
+    	    			ixx="0.0002825" ixy="0.0" ixz="0.0"
+    	    			iyy="0.002585" iyz="0.0"
+    	    			izz="0.002722"/>
 			</inertial>
 		</link>
