Commit message: Cleaned quadruped urdf

File: dtb_quadruped/dtb_quadruped_description/robots/dtb_quadruped.urdf.xacro (robot description, xacro)
@@ -1,7 +1,9 @@
 <?xml version="1.0"?>
 <robot xmlns:xacro = "http:://www.ros.org/wiki/xacro" name="dtb_quadruped">
+	<!--Xacro Properties-->
 	<xacro:property name="body_box_length" value="0.6"/>
 	<xacro:property name="body_box_width" value="0.25"/>
 	<xacro:property name="body_box_height" value="0.1"/>
+	<!-- Base Description-->
 	<link name="base_footprint"/>
 	<joint name="base_joint" type="fixed">
@@ -24,5 +26,4 @@
 				<box size = "${body_box_length} ${body_box_width} ${body_box_height}"/>
 			</geometry>
-			<material name = "body_color"/>
 		</collision>
 		<inertial>
@@ -35,4 +36,5 @@
 		</inertial>
 	</link>
+	<!-- Turn Motor -->
 	<xacro:macro name="t_motor_macro" params="t_motor_num x_pos y_pos">
 		<link name="t_motor_${t_motor_num}">
@@ -49,5 +51,4 @@
 					<cylinder length="0.03" radius="0.04"/>
 				</geometry>
-				<material name = "t_motor_color"/>
 			</collision>
 			<inertial>
@@ -71,4 +72,5 @@
 	<xacro:t_motor_macro t_motor_num="3" x_pos="${-(body_box_length/2)+0.016}" y_pos="1"/>
 	<xacro:t_motor_macro t_motor_num="4" x_pos="${-(body_box_length/2)+0.016}" y_pos="-1"/>
+	<!-- Turn to Loco Motor Joint -->
 	<xacro:macro name="t_l_link_macro" params="t_l_link_num">
 		<link name="t_l_link_${t_l_link_num}">
@@ -85,5 +87,4 @@
 					<cylinder length="0.08" radius="0.04"/>
 				</geometry>
-				<material name = "red"/>
 			</collision>
 			<inertial>
@@ -107,4 +108,5 @@
 	<xacro:t_l_link_macro t_l_link_num="3"/>
 	<xacro:t_l_link_macro t_l_link_num="4"/>
+	<!-- Loco Motor -->
 	<xacro:macro name="l_motor_macro" params="l_motor_num pose">
 		<link name="l_motor_${l_motor_num}">
@@ -121,5 +123,4 @@
 					<cylinder length="0.03" radius="0.039"/>
 				</geometry>
-				<material name = "l_motor_color"/>
 			</collision>
 			<inertial>
@@ -143,4 +144,5 @@
 	<xacro:l_motor_macro l_motor_num="3" pose="1"/>
 	<xacro:l_motor_macro l_motor_num="4" pose="-1"/>
+	<!-- Thigh Link -->
 	<xacro:macro name="thigh_link_macro" params="thigh_num pose">
 		<link name="thigh_link_${thigh_num}">
@@ -157,5 +159,4 @@
 					<box size="0.25 0.08 0.03"/>
 				</geometry>
-				<material name = "thigh_color"/>
 			</collision>
 			<inertial>
@@ -193,5 +194,4 @@
 					<cylinder length="0.03" radius="0.04"/>
 				</geometry>
-				<material name = "thigh_color"/>
 			</collision>
 			<inertial>
@@ -219,4 +219,5 @@
 	<xacro:thigh_semicirc_macro thigh_num="4" up_down="-1"/>
 	<xacro:thigh_semicirc_macro thigh_num="4" up_down="1"/>
+	<!-- Height Motor -->
 	<xacro:macro name="h_motor_macro" params="h_motor_num">
 		<link name="h_motor_${h_motor_num}">
@@ -233,5 +234,4 @@
 					<cylinder length="0.03" radius="0.041"/>
 				</geometry>
-				<material name = "h_motor_color"/>
 			</collision>
 			<inertial>
@@ -255,4 +255,5 @@
 	<xacro:h_motor_macro h_motor_num="3"/>
 	<xacro:h_motor_macro h_motor_num="4"/>
+	<!-- Calf Link -->
 	<xacro:macro name="calf_link_macro" params="calf_num">
 		<link name="calf_link_${calf_num}">
@@ -269,5 +270,4 @@
 					<box size="0.25 0.06 0.03"/>
 				</geometry>
-				<material name = "calf_color"/>
 			</collision>
 			<inertial>
@@ -305,5 +305,4 @@
 					<cylinder length="0.03" radius="0.03"/>
 				</geometry>
-				<material name = "calf_color"/>
 			</collision>
 			<inertial>
@@ -331,4 +330,5 @@
 	<xacro:calf_semicirc_macro calf_num="4" up_down="-1"/>
 	<xacro:calf_semicirc_macro calf_num="4" up_down="1"/>
+	<!-- Rviz Colors -->
 	<material name = "body_color">
 		<color rgba="1 1 1 1"/>

Commit message: Joints continuous to revolute

File: dtb_quadruped/dtb_quadruped_description/robots/dtb_quadruped.urdf.xacro (robot description, xacro)
@@ -5,4 +5,5 @@
 	<xacro:property name="body_box_width" value="0.25"/>
 	<xacro:property name="body_box_height" value="0.1"/>
+	<xacro:property name="M_PI" value="3.1415926"/>
 	<!-- Base Description-->
 	<link name="base_footprint"/>
@@ -61,9 +62,10 @@
 			</inertial>
 		</link>
-		<joint name="t_motor_${t_motor_num}_joint" type="continuous">
+		<joint name="t_motor_${t_motor_num}_joint" type="revolute">
 			<parent link="base_link"/>
 			<child link="t_motor_${t_motor_num}"/>
-			<origin xyz="${x_pos} ${((body_box_width/2)-0.03)*y_pos} ${(-body_box_height/2)+0.04}" rpy="0 1.5707 0"/>
-			<axis xyz="0 0 1"/>
+			<origin xyz="${x_pos} ${((body_box_width/2)-0.03)*y_pos} ${(-body_box_height/2)+0.04}" rpy="0 ${M_PI/2} 0"/>
+			<axis xyz="0 0 1"/>
+			<limit effort="15" lower="${(-M_PI/10)*y_pos}" upper="${(M_PI/10)*y_pos}" velocity="157"/>
 		</joint>
 	</xacro:macro>
@@ -133,9 +135,10 @@
 			</inertial>
 		</link>
-		<joint name="l_motor_${l_motor_num}_joint" type="continuous">
+		<joint name="l_motor_${l_motor_num}_joint" type="revolute">
 			<parent link="t_l_link_${l_motor_num}"/>
 			<child link="l_motor_${l_motor_num}"/>
-			<origin xyz="0 ${(0.055)*pose} 0" rpy="${(-1.5707)*pose} 0 0"/>
-			<axis xyz="0 0 1"/>
+			<origin xyz="0 ${(0.055)*pose} 0" rpy="${(-M_PI/2)*pose} 0 0"/>
+			<axis xyz="0 0 1"/>
+			<limit effort="15" lower="${(-M_PI/2)+((-M_PI/2)*pose)}" upper="${(M_PI/2)-((M_PI/2)*pose)}" velocity="157"/>
 		</joint>
 	</xacro:macro>
@@ -172,5 +175,5 @@
 			<parent link="l_motor_${thigh_num}"/>
 			<child link="thigh_link_${thigh_num}"/>
-			<origin xyz="0 ${0.125*pose} 0.015" rpy="0 0 ${1.5707*pose}"/>
+			<origin xyz="0 ${0.125*pose} 0.015" rpy="0 0 ${(M_PI/2)*pose}"/>
 			<axis xyz="0 0 1"/>
 		</joint>
@@ -220,5 +223,5 @@
 	<xacro:thigh_semicirc_macro thigh_num="4" up_down="1"/>
 	<!-- Height Motor -->
-	<xacro:macro name="h_motor_macro" params="h_motor_num">
+	<xacro:macro name="h_motor_macro" params="h_motor_num pose">
 		<link name="h_motor_${h_motor_num}">
 			<visual>
@@ -244,15 +247,16 @@
 			</inertial>
 		</link>
-		<joint name="h_motor_${h_motor_num}_joint" type="continuous">
+		<joint name="h_motor_${h_motor_num}_joint" type="revolute">
 			<parent link="thigh_link_${h_motor_num}"/>
 			<child link="h_motor_${h_motor_num}"/>
 			<origin xyz="0.125 0 0.015" rpy="0 0 0"/>
 			<axis xyz="0 0 1"/>
-		</joint>
-	</xacro:macro>
-	<xacro:h_motor_macro h_motor_num="1"/>
-	<xacro:h_motor_macro h_motor_num="2"/>
-	<xacro:h_motor_macro h_motor_num="3"/>
-	<xacro:h_motor_macro h_motor_num="4"/>
+			<limit effort="15" lower="${0 + (-M_PI*pose)}" upper="${M_PI-(pose*M_PI)}" velocity="157"/>
+		</joint>
+	</xacro:macro>
+	<xacro:h_motor_macro h_motor_num="1" pose="0"/>
+	<xacro:h_motor_macro h_motor_num="2" pose="1"/>
+	<xacro:h_motor_macro h_motor_num="3" pose="0"/>
+	<xacro:h_motor_macro h_motor_num="4" pose="1"/>
 	<!-- Calf Link -->
 	<xacro:macro name="calf_link_macro" params="calf_num">

Commit message: Changed motor effort

File: dtb_quadruped/dtb_quadruped_description/robots/dtb_quadruped.urdf.xacro (robot description, xacro)
@@ -6,5 +6,6 @@
 	<xacro:property name="body_box_width" value="0.25"/>
 	<xacro:property name="body_box_height" value="0.1"/>
-	<xacro:property name="M_PI" value="3.1415926"/>
+	<xacro:property name="M_PI" value="3.1415926535897931"/>
+	<xacro:property name="motor_effort" value="30"/>
 	<!-- Base Description-->
 	<link name="base_footprint"/>
@@ -68,5 +69,5 @@
 			<origin xyz="${x_pos} ${((body_box_width/2)-0.03)*y_pos} ${(-body_box_height/2)+0.04}" rpy="0 ${M_PI/2} 0"/>
 			<axis xyz="0 0 1"/>
-			<limit effort="15" lower="${(-M_PI/10)*y_pos}" upper="${(M_PI/10)*y_pos}" velocity="157"/>
+			<limit effort="${motor_effort}" lower="${(-M_PI/10)*y_pos}" upper="${(M_PI/10)*y_pos}" velocity="157"/>
 		</joint>
 	</xacro:macro>
@@ -141,5 +142,5 @@
 			<origin xyz="0 ${(0.055)*pose} 0" rpy="${(-M_PI/2)*pose} 0 0"/>
 			<axis xyz="0 0 1"/>
-			<limit effort="15" lower="${(-M_PI/2)+((-M_PI/2)*pose)}" upper="${(M_PI/2)-((M_PI/2)*pose)}" velocity="157"/>
+			<limit effort="${motor_effort}" lower="${(-M_PI/2)+((-M_PI/2)*pose)}" upper="${(M_PI/2)-((M_PI/2)*pose)}" velocity="157"/>
 		</joint>
 	</xacro:macro>
@@ -253,5 +254,5 @@
 			<origin xyz="0.125 0 0.015" rpy="0 0 0"/>
 			<axis xyz="0 0 1"/>
-			<limit effort="15" lower="${0 + (-M_PI*pose)}" upper="${M_PI-(pose*M_PI)}" velocity="157"/>
+			<limit effort="${motor_effort}" lower="${0 + (-M_PI*pose)}" upper="${M_PI-(pose*M_PI)}" velocity="157"/>
 		</joint>
 	</xacro:macro>

Commit message: Increased motor velocity

File: dtb_quadruped/dtb_quadruped_description/robots/dtb_quadruped.urdf.xacro (robot description, xacro)
@@ -8,5 +8,5 @@
 	<xacro:property name="M_PI" value="3.1415926"/>
 	<xacro:property name="motor_effort" value="50"/>
-	<xacro:property name="motor_velocity" value="${M_PI/2}"/>
+	<xacro:property name="motor_velocity" value="${M_PI}"/>
 	<!-- Base Description-->
 	<link name="base_footprint"/>
